Commit message: update package path

File: denso_robot_descriptions/vs087_description/vs087.urdf (robot description, URDF)
Before this commit: robot vs087, 8 links, 7 joints
Links:
- link J1: geometry collision mesh filename=package://denso_robot_descriptions/vs087_description/J1.dae scale=1 1 1; visual mesh filename=package://denso_robot_descriptions/vs087_description/J1.dae scale=1 1 1
- link J2: geometry collision mesh filename=package://denso_robot_descriptions/vs087_description/J2.dae scale=1 1 1; visual mesh filename=package://denso_robot_descriptions/vs087_description/J2.dae scale=1 1 1
- link J3: geometry collision mesh filename=package://denso_robot_descriptions/vs087_description/J3.dae scale=1 1 1; visual mesh filename=package://denso_robot_descriptions/vs087_description/J3.dae scale=1 1 1
- link J4: geometry collision mesh filename=package://denso_robot_descriptions/vs087_description/J4.dae scale=1 1 1; visual mesh filename=package://denso_robot_descriptions/vs087_description/J4.dae scale=1 1 1
- link J5: geometry collision mesh filename=package://denso_robot_descriptions/vs087_description/J5.dae scale=1 1 1; visual mesh filename=package://denso_robot_descriptions/vs087_description/J5.dae scale=1 1 1
- link J6: geometry collision mesh filename=package://denso_robot_descriptions/vs087_description/J6.dae scale=1 1 1; visual mesh filename=package://denso_robot_descriptions/vs087_description/J6.dae scale=1 1 1
- link base_link: geometry collision mesh filename=package://denso_robot_descriptions/vs087_description/base_l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 scale=1 1 1; visual mesh filename=package://denso_robot_descriptions/vs087_description/base_l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 scale=1 1 1

File: denso_robot_descriptions/vs087_description/vs087.urdf.xacro (robot description, xacro)
@@ -6,5 +6,5 @@
                 <origin xyz="0 0 0" rpy="0 0 0" />
                 <geometry>
-                    <mesh filename="package://vs087_description/J${num}.dae" scale="1 1 1" />
+                    <mesh filename="package://denso_robot_descriptions/vs087_description/J${num}.dae" scale="1 1 1" />
                 </geometry>
             </visual>
@@ -12,5 +12,5 @@
                 <origin xyz="0 0 0" rpy="0 0 0" />
                 <geometry>
-                    <mesh filename="package://vs087_description/J${num}.dae" scale="1 1 1" />
+                    <mesh filename="package://denso_robot_descriptions/vs087_description/J${num}.dae" scale="1 1 1" />
                 </geometry>
             </collision>
@@ -98,5 +98,5 @@
                 <origin rpy="0 0 0" xyz="0 0 0" />
                 <geometry>
-                    <mesh filename="package://vs087_description/base_link.dae" scale="1 1 1" />
+                    <mesh filename="package://denso_robot_descriptions/vs087_description/base_link.dae" scale="1 1 1" />
                 </geometry>
             </visual>
@@ -104,5 +104,5 @@
                 <origin rpy="0 0 0" xyz="0 0 0" />
                 <geometry>
-                    <mesh filename="package://vs087_description/base_link.dae" scale="1 1 1" />
+                    <mesh filename="package://denso_robot_descriptions/vs087_description/base_link.dae" scale="1 1 1" />
                 </geometry>
             </collision>
